File: minipcie-eth.sch (KiCad schematic (older format))
At the start: 7 parts, among them J1 UART2, J2 GPIO, U1 VoCore_v2

Commit message: Migrate to KiCad 5.1 :)
Parts:
- D2, D3, D9: symbol LED_Small_ALT -> device1:LED_Small_ALT
- J1: symbol Conn_01x04 -> minipcie-eth-rescue:Conn_01x04
- J2: symbol Conn_02x08_Odd_Even -> minipcie-eth-rescue:Conn_02x08_Odd_Even
- RN1: symbol R_Network04 -> device1:R_Network04
- U1: symbol VoCore_v2 -> win:VoCore_v2
Connections:
- net GND: no longer U1.19 (GND)
- net sdcard/SD_CLK: no longer names the net of U1.22 (SD_CLK)
- net sdcard/SD_CMD: no longer names the net of U1.23 (SD_CMD)
- net sdcard/SD_D0: no longer names the net of U1.21 (SD_D0)
- net sdcard/SD_D1: no longer names the net of U1.20 (SD_D1)
- net sdcard/SD_D2: no longer names the net of U1.25 (SD_D2)
- net sdcard/SD_D3: no longer names the net of U1.24 (SD_D3)
- no-connect marks 20 -> 27
Other:
- note removed: "XXX: Can we just avoid having to use external SD \ncard by compiling small enough OpenWRT \nthat just fits inside the VoCore2 memory?\n\nLess power consumption and less filesystem errors.\n\nAlternatively, use read read-only filesystem \nand switch off power to it via mosfet+gpio or simple PMIC."
Changed lines of the file:
@@
-EESchema Schematic File Version 3
-LIBS:power
-LIBS:device
-LIBS:transistors
-LIBS:conn
-LIBS:linear
-LIBS:regul
-LIBS:74xx
-LIBS:cmos4000
-LIBS:adc-dac
-LIBS:memory
-LIBS:xilinx
-LIBS:microcontrollers
-LIBS:dsp
-LIBS:microchip
-LIBS:analog_switches
-LIBS:motorola
-LIBS:texas
-LIBS:intel
-LIBS:audio
-LIBS:interface
-LIBS:digital-audio
-LIBS:philips
-LIBS:display
-LIBS:cypress
-LIBS:siliconi
-LIBS:opto
-LIBS:atmel
-LIBS:contrib
-LIBS:valves
-LIBS:win
-LIBS:freetronics_schematic
-LIBS:mpcie
-LIBS:si3406
-LIBS:si3404
-LIBS:SI-52003-F
-LIBS:ap2112
+EESchema Schematic File Version 4
 LIBS:minipcie-eth-cache
-EELAYER 26 0
+EELAYER 29 0
 EELAYER END
 $Descr A4 11693 8268
 encoding utf-8
-Sheet 1 4
+Sheet 1 3
 Title ""
 Date ""
@@
 $EndDescr
 $Comp
-L VoCore_v2 U1
+L win:VoCore_v2 U1
 U 1 1 5BAF0D89
 P 5710 3930
@@
 $EndSheet
 $Comp
-L Conn_01x04 J1
+L minipcie-eth-rescue:Conn_01x04 J1
 U 1 1 5BAF1493
 P 3770 4370
@@
 $EndComp
 $Comp
-L GND #PWR01
+L power1:GND #PWR01
 U 1 1 5BAF1546
 P 6520 5530
@@
 $EndComp
 $Comp
-L GND #PWR02
-U 1 1 5BAF157A
-P 5060 5380
-F 0 "#PWR02" H 5060 5130 50  0001 C CNN
-F 1 "GND" V 5065 5252 50  0000 R CNN
-F 2 "" H 5060 5380 50  0001 C CNN
-F 3 "" H 5060 5380 50  0001 C CNN
-	1    5060 5380
-	0    1    1    0
-$EndComp
-$Comp
-L GND #PWR03
+L power1:GND #PWR03
 U 1 1 5BAF158B
 P 8120 4740
@@
 $EndComp
 $Comp
-L GND #PWR04
+L power1:GND #PWR04
 U 1 1 5BAF15B1
 P 4830 2440
@@
 $EndComp
 $Comp
-L +5V #PWR05
+L power1:+5V #PWR05
 U 1 1 5BAF166D
 P 6160 5530
@@
 NoConn ~ 7160 4630
 $Comp
-L Conn_02x08_Odd_Even J2
+L minipcie-eth-rescue:Conn_02x08_Odd_Even J2
 U 1 1 5BAF1E64
 P 8630 4030
@@
 $EndComp
 $Comp
-L +5V #PWR06
+L power1:+5V #PWR06
 U 1 1 5BAF2AC1
 P 3970 4470
@@
 $EndComp
 $Comp
-L GND #PWR07
+L power1:GND #PWR07
 U 1 1 5BAF2AD4
 P 3970 4170
@@
 	6160 5380 6160 5530
 Wire Wire Line
-	6260 5380 6520 5380
+	6260 5380 6360 5380
 Wire Wire Line
 	6520 5380 6520 5530
 Connection ~ 6360 5380
 Wire Wire Line
-	5160 2300 5160 2480
+	5160 2300 5160 2390
 Wire Wire Line
 	5160 2390 4830 2390
@@
 	4830 2390 4830 2440
 Wire Wire Line
-	7160 4430 7160 4530
-Wire Wire Line
-	7270 4530 8240 4530
+	7160 4430 7160 4480
+Wire Wire Line
+	7270 4530 8120 4530
 Wire Wire Line
 	8240 4530 8240 4610
 Wire Wire Line
-	8240 4610 9050 4610
+	8240 4610 8930 4610
 Wire Wire Line
 	8930 4610 8930 4430
@@
 	8430 3930 8120 3930
 Wire Wire Line
-	8120 3930 8120 4740
+	8120 3930 8120 4530
 Connection ~ 8120 4530
 Wire Wire Line
@@
 	9050 4330 8930 4330
 Wire Wire Line
-	9050 4610 9050 4030
+	9050 4610 9050 4330
 Connection ~ 8930 4610
 Wire Wire Line
@@
 	5860 5380 5860 5950
 Wire Wire Line
-	5660 5610 5660 5380
-Wire Wire Line
-	2160 5610 5660 5610
-Wire Wire Line
-	5560 5690 5560 5380
-Wire Wire Line
-	2160 5690 5560 5690
-Wire Wire Line
-	5460 6010 5460 5380
-Wire Wire Line
-	2160 6010 5460 6010
-Wire Wire Line
-	5360 5920 5360 5380
-Wire Wire Line
-	2160 5920 5360 5920
-Wire Wire Line
-	5260 5450 5260 5380
-Wire Wire Line
-	2160 5450 5260 5450
-Wire Wire Line
-	5160 5530 5160 5380
-Wire Wire Line
-	2160 5530 5160 5530
-Wire Wire Line
 	2700 3480 4260 3480
 Wire Wire Line
@@
 Wire Wire Line
 	6560 2230 6560 1870
-Text Notes 1440 7310 0    60   ~ 0
-XXX: Can we just avoid having to use external SD \ncard by compiling small enough OpenWRT \nthat just fits inside the VoCore2 memory?\n\nLess power consumption and less filesystem errors.\n\nAlternatively, use read read-only filesystem \nand switch off power to it via mosfet+gpio or simple PMIC.
 Text Notes 7580 2490 0    60   ~ 0
 XXX: Review reset state for those two lines.\npull-up/pull-down accordingly.
 $Comp
-L LED_Small_ALT D9
+L device1:LED_Small_ALT D9
 U 1 1 5BB77A38
 P 3480 2400
@@
 $EndComp
 $Comp
-L LED_Small_ALT D2
+L device1:LED_Small_ALT D2
 U 1 1 5BB77A74
 P 3740 2390
@@
 $EndComp
 $Comp
-L LED_Small_ALT D3
+L device1:LED_Small_ALT D3
 U 1 1 5BB77AA6
 P 3990 2400
@@
 $EndComp
 $Comp
-L R_Network04 RN1
+L device1:R_Network04 RN1
 U 1 1 5BB77E7E
 P 3580 2830
@@
 $EndComp
 $Comp
-L GND #PWR08
+L power1:GND #PWR08
 U 1 1 5BB7822B
 P 3780 3030
@@
 Connection ~ 7160 4480
 $Comp
-L GND #PWR09
+L power1:GND #PWR09
 U 1 1 5BC0D564
 P 7300 3040
@@
 (C) Roman Valls Guimera (brainstorm at nopcode dot org)
 $Comp
-L GND #PWR010
+L power1:GND #PWR010
 U 1 1 5BC3827A
 P 1690 4410
@@
 	1690 4210 1690 4120
 $Comp
-L +5V #PWR011
+L power1:+5V #PWR011
 U 1 1 5BC389B7
 P 1690 4120
@@
 $EndComp
 $Comp
-L GND #PWR012
+L power1:GND #PWR012
 U 1 1 5BC444DB
 P 1700 3510
@@
 ETH_INGRESS_LED
 $Comp
-L +3V3 #PWR013
+L power1:+3V3 #PWR013
 U 1 1 5BC46C2B
 P 1700 3140
@@
 $EndComp
 $Comp
-L +3V3 #PWR014
+L power1:+3V3 #PWR014
 U 1 1 5BC46E95
 P 4190 1950
@@
 Text Notes 630  2740 0    60   ~ 0
 XXX: Add decoupling caps on power rails as shown in\nlaf0rge minipcie schematic:\n\nhttps://osmocom.org/projects/mpcie-breakout/wiki
-$Sheet
-S 1440 5320 720  1060
-U 5BAF0F57
-F0 "sdcard" 60
-F1 "sdcard.sch" 60
-F2 "SD_D0" I R 2160 5450 60
-F3 "SD_D1" I R 2160 5530 60
-F4 "SD_D2" I R 2160 5610 60
-F5 "SD_D3" I R 2160 5690 60
-F6 "SD_CMD" I R 2160 6010 60
-F7 "SD_CLK" I R 2160 5920 60
-F8 "SD_VDD" I R 2160 6260 60
-$EndSheet
-$Comp
-L +3V3 #PWR015
-U 1 1 5BC5E4DC
-P 2280 6260
-F 0 "#PWR015" H 2280 6110 50  0001 C CNN
-F 1 "+3V3" H 2295 6433 50  0000 C CNN
-F 2 "" H 2280 6260 50  0001 C CNN
-F 3 "" H 2280 6260 50  0001 C CNN
-	1    2280 6260
-	1    0    0    -1
-$EndComp
-Wire Wire Line
-	2160 6260 2280 6260
+NoConn ~ 5660 5380
+NoConn ~ 5560 5380
+NoConn ~ 5460 5380
+NoConn ~ 5360 5380
+NoConn ~ 5260 5380
+NoConn ~ 5160 5380
+NoConn ~ 5060 5380
+Wire Wire Line
+	6360 5380 6520 5380
+Wire Wire Line
+	8120 4530 8180 4530
+Wire Wire Line
+	8120 4530 8120 4740
+Wire Wire Line
+	8180 4530 8240 4530
+Wire Wire Line
+	8930 4610 9050 4610
+Wire Wire Line
+	9050 4330 9050 4230
+Wire Wire Line
+	9050 4230 9050 4130
+Wire Wire Line
+	9050 4130 9050 4030
+Wire Wire Line
+	5160 2390 5160 2480
+Wire Wire Line
+	7160 4480 7160 4530
 $EndSCHEMATC
