File: minipcie.sch (KiCad schematic (older format))
At the start: 1 part, among them U4 MPCIE-Socket

Commit message: Move libs away from rescue. Re-constrained board layout since cutouts were not perpendicular (overconstrained)
Parts:
- U4: symbol minipcie-eth-rescue:MPCIE-Socket-mpcie -> minipcie-eth-rescue:MPCIE-Socket-mpcie-minipcie-eth-rescue-minipcie-eth-rescue
Changed lines of the file:
@@
 $EndDescr
 $Comp
-L minipcie-eth-rescue:MPCIE-Socket-mpcie U4
+L minipcie-eth-rescue:MPCIE-Socket-mpcie-minipcie-eth-rescue-minipcie-eth-rescue U4
 U 1 1 5BB36495
 P 3940 4080
+AR Path="/5BB36495" Ref="U4"  Part="1"
+AR Path="/5BAF0FB4/5BB36495" Ref="U4"  Part="1"
 F 0 "U4" H 3940 5517 60  0000 C CNN
 F 1 "MPCIE-Socket" H 3940 5411 60  0000 C CNN
